File: EWP Control.kicad_sch (KiCad schematic)
At the start: 93 parts, among them Q1 SQJ411EP-T1_GE3, SW1 HX 3X4X2.5-PA-4N PUSH BUTTON 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, U1 RP2350B_C42415655, U10 BME280, U11 DS3231MZ+, U12 INA226AIDGSR, U13 TPL5010DDCR, U14 BTS50015-1TAD, U15 BTS50015-1TAD, U2 ESP32-S3, U3 W25Q128JVSIQTR, U4 MT25QL01GBBB8ESF-0SIT TR, U5 APS51208N-OBR-BD, U6 AD7124-8BCPZ, U7 AD5689RBRUZ, U8 TPS54540DDAR, U9 TLV75533PDBVR, X1 X49SM12MSD2SI, X2 X49SM12MSD2SI, X3 HSO531S 12MHZ 1.6~3.6V, X4 40MHZ/3225/12PF/10PPM

Commit message: Close: 5 files changed EWP Control.kicad_pcb 4102/0/0 EWP Control.kicad_prl 105/0/0 EWP Control.kicad_pro 13/0/0 EWP Control.kicad_sch 0/36947/10534 fp-lib-table 9/0/0
Connections:
- net +3V3: now also C33.1, U9.5 (OUT); no longer C8.2
- net VDD: no longer C7.1, L1.2, L2.2, U1.32 (DVDD), U1.51 (DVDD), U1.65 (VREG_FB)
- new net 1v1: C7.1, L1.2, L2.2, U1.51 (DVDD), U1.65 (VREG_FB)
- no-connect marks 0 -> 12
