File: EWP Control.kicad_sch (KiCad schematic)
At the start: 111 parts, among them CN1 5557-2P Straight line 2*1P, Q1 SQJ411EP-T1_GE3, SW1 HX 3X4X2.5-PA-4N PUSH BUTTON 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, U1 RP2350B_C42415655, U10 BME280, U11 DS3231MZ+, U12 INA226AIDGSR, U13 TPL5010DDCR, U14 BTS50015-1TAD, U15 BTS50015-1TAD, U16 USB_C_RECEPTACLE_HRO_TYPE-C-3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, U2 ESP32-S3, U3 W25Q128JVSIQTR, U4 MT25QL01GBBB8ESF-0SIT TR, U5 APS51208N-OBR-BD, U6 AD7124-8BCPZ, U7 AD5689RBRUZ, U8 TPS54540DDAR, U9 TLV75533PDBVR, X1 X49SM12MSD2SI, X2 X49SM12MSD2SI, X4 40MHZ/3225/12PF/10PPM

Commit message: Complete schematic circuit design + 4-layer PCB structure/zones/basic routing
Schematic (EWP Control.kicad_sch):
- Full netlist design for all 16 ICs + 55 caps + 32 resistors + crystals/
  inductors/diodes/MOSFET/switch/connectors via tools/fix_schematic.py
- 527 local labels define 96 nets; 106 no_connects for unused pins;
  13 PWR_FLAG symbols drive all power nets (ERC pin_not_connected=0,
  power_pin_not_driven=0)
- 0 floating pins across all 697 component pins (was 697 floating)
- Each pin->net traceable to factory_config.h (ESP32-S3) or P01-P15 page
  plan (RP2350B/ADC/DAC/power/sensors/actuators)
- GPIO48 (absent on ESP32-S3 QFN-56) -> RGB moved to GPIO38 (pin 43)

PCB (EWP Control.kicad_pcb):
- 4-layer stack: F.Cu / In1.Cu(GND) / In2.Cu(PWR) / B.Cu (was 2-layer)
- Board outline compacted 170x130 -> 78x66 mm
- 4 copper zones: GND full-board on In1.Cu; +3.3V/+5V/VBAT on In2.Cu
- 216 trace items: 137 segments (SPI/I2C/UART/QSPI buses) + 79 power vias
  tying every IC power pad to inner planes
- Pad netlist re-annotated from fresh schematic (92 nets on pads)

Firmware:
- SC_FACTORY_PIN_RGB 48 -> 38 (matches QFN-56 pin 43)
- verify_release.py: release_static_gate = ok
- verify_control_math.py: 94.7% steady quality
Connections:
- net 1v1 is gone; now on net +3V3: C7.1, L1.2, U1.10 (DVDD), U1.32 (DVDD), U1.51 (DVDD), U1.65 (VREG_FB)
- net 3V3_TARGET_SENSE is gone; now on net +3V3: R12.1, R17.1
- net ADC_CS is gone; now on net +3V3: Card1.7 (DAT0), U1.16 (GPIO16), U6.32 (~{CS})
- net ADC_MISO is gone; now on net +3V3: Card1.5 (CLK), U1.18 (GPIO18), U13.5 (WAKE), U6.28 (DOUT/~{RDY})
- net ADC_SCLK is gone; now on net +3V3: Card1.8 (DAT1), U1.17 (GPIO17), U13.4 (DONE), U6.30 (SCLK)
- net BME_CSB is gone; now on net +3V3: R20.2, R9.1, U10.2 (CSB)
- net BOOT_BUTTON is gone; now on net +3V3: C55.1, D1.2 (A), R2.2, SW1.1, SW1.2, U13.6 (RSTn), U2.4 (CHIP_PU)
- net DAC_SYNC is gone; now on net +3V3: U1.55 (GPIO44_ADC4), U7.13 (~{SYNC})
- net ESP_GPIO0_BOOT is gone; now on net +3V3: D1.1 (K), U2.5 (GPIO0)
- net ESP_UART0_RXD is gone; now on net +3V3: U1.77 (GPIO0), U2.50 (U0RXD)
- net HS_SW1_EN is gone; now on net +3V3: R22.1, U14.2 (IN)
- net HS_SW1_IS is gone; now on net +3V3: R10.1, R15.1, R16.2, R19.1, R31.1, U12.3 (Alert), U14.3 (IS)
- net HS_SW2_EN is gone; now on net +3V3: Card1.2 (CD/DAT3), U1.21 (GPIO21), U15.2 (IN)
- net HS_SW2_IS is gone; now on net +3V3: R11.1, R23.1, R32.1, U15.3 (IS)
- net I2C_SCL is gone; now on net +3V3: U10.4 (SCK), U11.8 (SCL), U12.5 (SCL)
- net I2C_SDA is gone; now on net +3V3: U10.3 (SDI), U11.7 (SDA), U12.4 (SDA)
- net MCU_RUN is gone; now on net +3V3: R25.2, U1.35 (RUN)
- net N_U8_BOOT is gone; now on net +3V3: C25.1, U8.1 (BOOT)
- net N_U8_COMP is gone; now on net +3V3: C27.1, C28.1, U8.6 (COMP)
- net N_U8_COMP_S is gone; now on net +3V3: C27.2, R8.1
- net N_U8_FB is gone; now on net +3V3: R5.2, R6.1, U8.5 (FB)
- net N_U8_RT is gone; now on net +3V3: R7.1, U8.4 (RT/CLK)
- net PSRAM_CE is gone; now on net +3V3: R18.2, R28.1, U1.44 (GPIO35), U5.A3 (~{CE})
- net PSRAM_CLK is gone; now on net +3V3: U1.43 (GPIO34), U5.B2 (CLK)
- net PSRAM_DQ0 is gone; now on net DAC_SCLK: U1.42 (GPIO33), U5.D3 (ADQ0)
- net PSRAM_DQ2 is gone; now on net +3V3: U1.39 (GPIO31), U5.C4 (ADQ2)
- net PSRAM_DQ3 is gone; now on net +3V3: U1.38 (GPIO30), U5.D4 (ADQ3)
- net PSRAM_DQ4 is gone; now on net +3V3: U1.37 (GPIO29), U5.D5 (ADQ4)
- net PSRAM_DQ5 is gone; now on net +3V3: U1.36 (GPIO28), U5.E3 (ADQ5)
- net PSRAM_DQ6 is gone; now on net ESP_UART0_TXD: R1.1, U5.E2 (ADQ6)
- net PSRAM_DQ7 is gone; now on net +3V3: U1.34 (SWDIO), U5.E1 (ADQ7)
- net PSRAM_DQS is gone; now on net +3V3: U1.45 (GPIO36), U5.C3 (DQS/DM)
- net PSRAM_RST is gone; now on net +3V3: R29.1, U1.46 (GPIO37), U5.A4 (~{RST})
- net PWR_OUT1 is gone; now on net +3V3: U14.5 (OUT), U14.6 (OUT), U14.7 (OUT)
- net PWR_OUT2 is gone; now on net +3V3: U15.5 (OUT), U15.6 (OUT), U15.7 (OUT)
- net QSPI1_CS is gone; now on net +3V3: U1.13 (GPIO14), U4.7 (~{S})
- net QSPI1_IO0 is gone; now on net +3V3: U1.8 (GPIO10), U4.15 (DQ0)
- net QSPI1_IO1 is gone; now on net +3V3: U1.9 (GPIO11), U4.8 (DQ1)
- net QSPI1_IO3 is gone; now on net ESP_UART0_TXD: U1.11 (GPIO12), U4.1 (DQ3/~{HOLD})
- net QSPI1_SCLK is gone; now on net +3V3: U1.12 (GPIO13), U4.16 (C)
- net QSPI_SD0 is gone; now on net +3V3: U1.72 (QSPI_SD0), U3.5 (DI)
- net QSPI_SD1 is gone; now on net +3V3: U1.74 (QSPI_SD1), U3.2 (DO)
- net QSPI_SD2 is gone; now on net +3V3: U1.73 (QSPI_SD2), U3.3 (IO2)
- net QSPI_SD3 is gone; now on net QSPI_SCLK: U1.70 (QSPI_SD3), U3.7 (IO3)
- net QSPI_SS is gone; now on net +3V3: U1.75 (QSPI_SS), U3.1 (~{CS})
- net REGCAPA is gone; now on net +3V3: C12.1, U6.24 (REGCAPA)
- net RP_SWCLK is gone; now on net +3V3: CN1.1, U1.33 (SWCLK)
- net SD_CD is gone; now on net +3V3: Card1.SW1, R3.1, U1.22 (GPIO22)
- net SD_DAT2 is gone; now on net +3V3: Card1.1 (DAT2), U1.20 (GPIO20)
- net SER_R30_A is gone; now on net +3V3: R30.1, U13.3 (DELAY/M_RST)
- net U2_XTAL_N is gone; now on net +3V3: U2.53 (XTAL_N), X4.3
- net USB_CON_N is gone; now on net +3V3: R26.2, U16.A7 (DN1), U16.B7 (DN2)
- net USB_CON_P is gone; now on net +3V3: R27.2, U16.A6 (DP1), U16.B6 (DP2)
- net USB_D_N is gone; now on net +3V3: R26.1, U1.66 (USB_DM)
- net USB_D_P is gone; now on net +3V3: R27.1, U1.67 (USB_DP)
- net VBAT is gone; now on net +3V3: C36.1, R24.1, U11.6 (VBAT), U12.10 (VIN+), U12.8 (VBUS), U14.8 (VS), U15.8 (VS)
- net VBAT_LOAD is gone; now on net +3V3: R24.2, U12.9 (VIN-)
- net VBUS is gone; now on net +3V3: U16.A4B9 (VBUS), U16.B4A9 (VBUS)
- net VIN is gone; now on net +3V3: Q1.5 (D)
- net VOUT_SENSE is gone; now on net +3V3: R5.1
- net VSW is gone; now on net +3V3: C25.2, U8.8 (SW)
- net VSYS is gone; now on net +3V3: C32.1, Q1.1 (S), Q1.2 (S), Q1.3 (S), R14.1, U9.1 (IN)
- net +3V3: now also C13.1, C24.1, C52.1, C52.2, C53.1, C53.2, Card1.11, Card1.12, R13.2, R14.2, R4.1, R4.2, U1.25 (GPIO24), U1.27 (GPIO26), U1.28 (GPIO27), U16.17, U16.18, U16.19, U16.20, U16.A5 (CC1), U16.A8 (SBU1), U16.B5 (CC2), U16.B8 (SBU2), U2.10 (GPIO5), U2.13 (GPIO8), U2.16 (GPIO11), U2.17 (GPIO12), U2.18 (GPIO13), U2.24 (GPIO18), U2.25 (GPIO19), U2.26 (GPIO20), U2.27 (GPIO21), U2.28 (SPICS1), U2.30 (SPIHD), U2.31 (SPIWP), U2.34 (SPIQ), U2.35 (SPID), U2.38 (GPIO33), U2.41 (GPIO36), U2.51 (GPIO45), U2.52 (GPIO46), U2.7 (GPIO2), U4.6 (DNU), U5.B3 (NC), U5.C2 (RFU), U5.C5 (NC), U6.1 (REGCAPD), U6.11 (AIN7/IOUT/VBIAS), U6.12 (REFIN+), U6.13 (REFIN-), U6.14 (AIN8/IOUT/VBIAS), U6.15 (AIN9/IOUT/VBIAS), U6.16 (AIN10/IOUT/VBIAS), U6.18 (AIN12/IOUT/VBIAS), U6.19 (AIN13/IOUT/VBIAS), U6.20 (AIN14/IOUT/VBIAS/REFIN2(+)), U6.21 (AIN15/IOUT/VBIAS/REFIN2(–)), U6.22 (REFOUT), U6.25 (PSW), U6.5 (AIN1/IOUT/VBIAS), U6.9 (AIN5/IOUT/VBIAS/P4), U8.2 (VIN), U8.3 (EN), U9.3 (EN), U9.4 (NC)
- net DAC_SDO: now also U6.6 (AIN2/IOUT/VBIAS/P1)
- net ESP_UART0_TXD: now also U1.26 (GPIO25)
- net SD_MISO: now reaches U2.12 (GPIO7)
- net SD_MOSI: now reaches U2.15 (GPIO10)
- net ECU_REQUEST: now reaches U2.19 (GPIO14)
- net FAN_PWM: now reaches U2.21 (XTAL_32K_P)
- net PUMP_PWM: now reaches U2.22 (XTAL_32K_N)
- net PUMP_SSR: now reaches U2.23 (GPIO17)
- net DAC_VOUTB: now reaches U7.2 (NC)
- net DAC_VOUTA: now reaches U7.6 (NC)
- net V5V_SENSE: now reaches U6.10 (AIN6/IOUT/VBIAS)
- no-connect marks 12 -> 106
